File: Hardware/Qwiic/SparkFun_6DoF_LSM6DSV16X.brd (EAGLE design)
At the start: 25.4 x 25.4 mm, 68 parts, among them J1 QWIIC_RIGHT_ANGLE, J2 QWIIC_RIGHT_ANGLE, U2 LSM6DSV16X

Commit message: Approves air wires, shuffles schematic
Routing:
- net SCL: track 38.7 -> 40.4 mm
- net OCS: track 21.3 -> 22.3 mm
- net POCI_AUX: track 25.0 -> 25.8 mm
Changed lines of the file:
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@@
 <wire x1="13.843" y1="6.731" x2="13.843" y2="1.397" width="0.254" layer="1"/>
 <contactref element="U2" pad="P13"/>
-<wire x1="12.7" y1="10.3284" x2="12.7" y2="11.7" width="0" layer="19" extent="1-1"/>
+<wire x1="12.74445" y1="9.994" x2="12.7" y2="10.03845" width="0.254" layer="1"/>
+<wire x1="12.7" y1="10.03845" x2="12.7" y2="11.7" width="0.254" layer="1"/>
 </signal>
 <signal name="SDA/PICO">
@@
 <signal name="INT2">
 <contactref element="JP3" pad="1"/>
-<wire x1="11.43" y1="12.95" x2="10.537" y2="12.95" width="0.254" layer="1"/>
 <via x="7.239" y="12.573" extent="1-16" drill="0.3"/>
 <wire x1="7.239" y1="12.573" x2="7.239" y2="13.858" width="0.254" layer="16"/>
@@
 <wire x1="10.537" y1="12.95" x2="10.16" y2="12.573" width="0.254" layer="1"/>
 <contactref element="U2" pad="P9"/>
-<wire x1="11.43" y1="12.95" x2="11.5375" y2="12.95" width="0" layer="19" extent="1-1"/>
+<wire x1="11.5375" y1="12.95" x2="10.537" y2="12.95" width="0.254" layer="1"/>
 </signal>
 <signal name="3.3V">
@@
 <wire x1="10.06621875" y1="11.9404" x2="10.57581875" y2="12.45" width="0.254" layer="1"/>
 <contactref element="U2" pad="P10"/>
-<wire x1="10.57581875" y1="12.45" x2="11.5375" y2="12.45" width="0" layer="19" extent="1-1"/>
+<wire x1="10.57581875" y1="12.45" x2="11.5375" y2="12.45" width="0.254" layer="1"/>
 </signal>
 <signal name="N$5">
@@
 <contactref element="JP3" pad="6"/>
 <via x="8.636" y="11.4094" extent="1-16" drill="0.3"/>
-<wire x1="10.7416375" y1="11.95" x2="10.2240375" y2="11.4324" width="0.254" layer="1"/>
+<wire x1="10.2240375" y1="11.4324" x2="10.7416375" y2="11.95" width="0.254" layer="1"/>
 <wire x1="8.659" y1="11.4324" x2="8.636" y2="11.4094" width="0.254" layer="1"/>
 <wire x1="10.2240375" y1="11.4324" x2="8.659" y2="11.4324" width="0.254" layer="1"/>
@@
 <wire x1="17.6784" y1="17.5514" x2="19.05" y2="18.923" width="0.254" layer="1"/>
 <contactref element="U2" pad="P11"/>
-<wire x1="10.7416375" y1="11.95" x2="11.5375" y2="11.95" width="0" layer="19" extent="1-1"/>
+<wire x1="10.7416375" y1="11.95" x2="11.5375" y2="11.95" width="0.254" layer="1"/>
 </signal>
 <signal name="N$7">
