File: Hardware/Qwiic/Qwiic Board with Filter/SparkFun_6DoF_LSM6DSV16X.brd (EAGLE design)
At the start: 25.4 x 25.4 mm, 87 parts, among them J1 QWIIC_RIGHT_ANGLE, J2 QWIIC_RIGHT_ANGLE, U2 LSM6DSV16X

Commit message: Changes version to v01, fixes air wires
Other:
- board text added: "v01"
- board text removed: "v10"
Changed lines of the file:
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@@
 <wire x1="0" y1="0" x2="25.4" y2="0" width="0.2032" layer="20"/>
 <wire x1="25.4" y1="0" x2="25.4" y2="25.4" width="0.2032" layer="20"/>
-<text x="24.139525" y="11.420475" size="0.8128" layer="16" font="vector" ratio="22" rot="MR90">v10</text>
+<text x="24.139525" y="11.420475" size="0.8128" layer="16" font="vector" ratio="22" rot="MR90">v01</text>
 <wire x1="0.3302" y1="7.546975" x2="2.2352" y2="7.546975" width="0.254" layer="21"/>
 <wire x1="1.7272" y1="7.038975" x2="1.7272" y2="8.181975" width="0.254" layer="21" curve="-180"/>
@@
 <via x="16.1036" y="10.3378" extent="1-16" drill="0.3"/>
 <via x="15.1638" y="23.0886" extent="1-16" drill="0.3"/>
-<wire x1="11.85" y1="15.201" x2="11.85" y2="15.24" width="0.254" layer="1"/>
 <wire x1="12.7" y1="14.39" x2="12.529" y2="14.561" width="0.254" layer="1"/>
 <wire x1="12.529" y1="14.561" x2="11.85" y2="15.24" width="0.254" layer="1"/>
@@
 <wire x1="3.81" y1="10.541" x2="4.191" y2="10.16" width="0.254" layer="1"/>
 <wire x1="7.747" y1="9.525" x2="7.747" y2="6.985" width="0.254" layer="1"/>
-<wire x1="16.002" y1="9.398" x2="15.406" y2="9.994" width="0.254" layer="1"/>
+<wire x1="15.406" y1="9.994" x2="16.002" y2="9.398" width="0.254" layer="1"/>
 <via x="16.002" y="8.5066" extent="1-16" drill="0.3"/>
 <wire x1="7.747" y1="6.985" x2="8.5598" y2="6.1722" width="0.254" layer="1"/>
@@
 <wire x1="14.732" y1="10.922" x2="15.748" y2="10.922" width="0.254" layer="1"/>
 <wire x1="15.748" y1="10.922" x2="17.018" y2="12.192" width="0.254" layer="1"/>
-<wire x1="14.859" y1="10.287" x2="14.652175" y2="10.080175" width="0.254" layer="1"/>
 <wire x1="11.43" y1="5.207" x2="11.43" y2="1.27" width="0.254" layer="1"/>
 <via x="12.7762" y="6.0452" extent="1-16" drill="0.3"/>
@@
 <contactref element="U2" pad="P14"/>
 <wire x1="13.2" y1="11.311" x2="13.2" y2="11.7" width="0.254" layer="1"/>
-<wire x1="15.406" y1="9.994" x2="14.732" y2="9.994" width="0.254" layer="1"/>
-<wire x1="14.732" y1="9.994" x2="14.732" y2="10.922" width="0.254" layer="1"/>
 <wire x1="17.018" y1="12.192" x2="18.161" y2="12.192" width="0.254" layer="1"/>
 <wire x1="18.161" y1="12.192" x2="19.169" y2="13.2" width="0.254" layer="1"/>
@@
 <wire x1="12.7" y1="5.969" x2="12.7762" y2="6.0452" width="0.254" layer="1"/>
 <wire x1="12.7" y1="2.54" x2="12.7" y2="5.969" width="0.254" layer="1"/>
-<wire x1="14.732" y1="9.994" x2="14.652175" y2="10.080175" width="0" layer="19" extent="1-1"/>
+<wire x1="14.732" y1="9.994" x2="14.732" y2="10.922" width="0.254" layer="1"/>
+<wire x1="14.732" y1="9.994" x2="15.406" y2="9.994" width="0.254" layer="1"/>
 </signal>
 <signal name="!CS!">
@@
 <contactref element="JP1" pad="2"/>
 <wire x1="12.065" y1="11.049" x2="12.2" y2="11.184" width="0.254" layer="1"/>
-<wire x1="12.065" y1="11.049" x2="11.049" y2="11.049" width="0.254" layer="1"/>
-<wire x1="10.7442" y1="10.7442" x2="11.049" y2="11.049" width="0.254" layer="1"/>
+<wire x1="11.049" y1="11.049" x2="12.065" y2="11.049" width="0.254" layer="1"/>
 <via x="9.398" y="9.525" extent="1-16" drill="0.3"/>
 <wire x1="16.51" y1="1.27" x2="16.51" y2="2.794" width="0.254" layer="1"/>
@@
 <contactref element="U2" pad="P12"/>
 <wire x1="12.2" y1="11.184" x2="12.2" y2="11.7" width="0.254" layer="1"/>
-<wire x1="10.7442" y1="10.0829" x2="10.7442" y2="10.7442" width="0.254" layer="1"/>
+<wire x1="9.8797" y1="10.0067" x2="9.398" y2="9.525" width="0.254" layer="1"/>
+<wire x1="10.668" y1="10.0067" x2="10.668" y2="10.668" width="0.254" layer="1"/>
+<wire x1="10.668" y1="10.668" x2="11.049" y2="11.049" width="0.254" layer="1"/>
 <wire x1="10.668" y1="10.0067" x2="9.8797" y2="10.0067" width="0.254" layer="1"/>
-<wire x1="9.8797" y1="10.0067" x2="9.398" y2="9.525" width="0.254" layer="1"/>
-<wire x1="10.668" y1="10.0067" x2="10.7442" y2="10.0829" width="0" layer="19" extent="1-1"/>
 </signal>
 <signal name="POCI/SA0">
@@
 <wire x1="14.732" y1="16.891" x2="9.271" y2="16.891" width="0.254" layer="1"/>
 <wire x1="14.8306625" y1="12.95" x2="16.002" y2="14.1213375" width="0.254" layer="1"/>
-<wire x1="10.1473" y1="19.0373" x2="10.16" y2="19.05" width="0.254" layer="16"/>
 <wire x1="10.16" y1="19.05" x2="10.16" y2="16.8783" width="0.254" layer="16"/>
 <wire x1="10.16" y1="16.8783" x2="10.1473" y2="16.8656" width="0.254" layer="16"/>
