File: Hardware/Qwiic/Qwiic Board with Filter/SparkFun_6DoF_LSM6DSV16X.sch (EAGLE design)
At the start: 40 parts, among them J1 QWIIC_RIGHT_ANGLE, J2 QWIIC_RIGHT_ANGLE, U2 LSM6DSV16X

Commit message: Changes version to v01, fixes air wires
Other:
- note added: "v01"
- note removed: "v10"
Changed lines of the file:
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@@
 <text x="93.726" y="261.874" size="1.27" layer="97" font="vector">VDD Range: 1.71V - 3.6V
 VDDIO Range: 1.62V - 3.6V</text>
-<text x="421.64" y="7.62" size="2.54" layer="94" font="vector">v10</text>
+<text x="421.64" y="7.62" size="2.54" layer="94" font="vector">v01</text>
 <text x="325.12" y="271.78" size="2.54" layer="94" font="vector" align="center">Jumpers</text>
 <text x="340.36" y="213.36" size="1.778" layer="97" font="vector">Cut trace to
