File: Hardware/Qwiic/Basic Qwiic Board/SparkFun_6DoF_LSM6DSV16X.sch (EAGLE design)
At the start: 31 parts, among them J1 QWIIC_RIGHT_ANGLE, J2 QWIIC_RIGHT_ANGLE, U2 LSM6DSV16X

Commit message: Changes silk label on bottom to "SDX instead of "PICOX"
Connections:
- net PICO_AUX renamed SDX/PICO_AUX
Changed lines of the file:
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@@
 </segment>
 </net>
-<net name="PICO_AUX" class="0">
+<net name="SDX/PICO_AUX" class="0">
 <segment>
 <pinref part="JP3" gate="JP1" pin="5"/>
